Commit message: 4-16-2024

File: impact_urdf/urdf/output.urdf (robot description, URDF)
Before this commit: robot ar3, 15 links, 14 joints
Links:
- removed link image_calibration_link
- removed link impact_camera_calibration_base_link
- removed link impact_camera_calibration_link
- added link camera_color_frame
- added link camera_color_optical_frame
- added link camera_depth_frame
- added link camera_depth_optical_frame
- added link camera_left_ir_frame
- added link camera_left_ir_optical_frame
- added link camera_right_ir_frame
- added link camera_right_ir_optical_frame
- added link left_finger, mass 0.0454654477917792; collision box size=0.1 0.02 0.04; visual mesh filename=package://wheeltec_gripper_description/meshes/fingers.STL
- added link right_finger, mass 0.0454654472444149; collision box size=0.1 0.02 0.04; visual mesh filename=package://wheeltec_gripper_description/meshes/fingers.STL
- added link wheeltec_gripper_base_link
- added link wheeltec_gripper_center; visual box size=0.01 0.01 0.01
- added link wheeltec_gripper_chaise, mass 0.102600550272344; collision box size=0.05 0.08 0.045; visual mesh filename=package://wheeltec_gripper_description/meshes/gripperbase.S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
- link camera_link: mass 0.072 -> 0.564
Joints:
- removed joint image_link_joint
- removed joint impact_camera_calibration_base_link_joint
- removed joint impact_camera_calibration_end_link_joint
- added joint camera_color_joint: type fixed, parent camera_depth_frame, child camera_color_frame, origin xyz=0 0.015 0 rpy=0 0 0
- added joint camera_color_optical_joint: type fixed, parent camera_color_frame, child camera_color_optical_frame, origin xyz=0 0 0 rpy=-1.5707963267948966 0 -1.5707963267948966
- added joint camera_depth_joint: type fixed, parent camera_link, child camera_depth_frame, origin xyz=0 0 0 rpy=0 0 0
- added joint camera_depth_optical_joint: type fixed, parent camera_depth_frame, child camera_depth_optical_frame, origin xyz=0 0 0 rpy=-1.5707963267948966 0 -1.5707963267948966
- added joint camera_left_ir_joint: type fixed, parent camera_depth_frame, child camera_left_ir_frame, origin xyz=0 0.0 0 rpy=0 0 0
- added joint camera_left_ir_optical_joint: type fixed, parent camera_left_ir_frame, child camera_left_ir_optical_frame, origin xyz=0 0 0 rpy=-1.5707963267948966 0 -1.5707963267948966
- added joint camera_right_ir_joint: type fixed, parent camera_depth_frame, child camera_right_ir_frame, origin xyz=0 -0.05 0 rpy=0 0 0
- added joint camera_right_ir_optical_joint: type fixed, parent camera_right_ir_frame, child camera_right_ir_optical_frame, origin xyz=0 0 0 rpy=-1.5707963267948966 0 -1.5707963267948966
- added joint left_finger_joint: type revolute, parent wheeltec_gripper_chaise, child left_finger, origin xyz=0.071508 -0.024545 -0.020131 rpy=0 0 0, axis 2.5729E-05 -0.080001 0.99679, limit lower=0 upper=0.7298 effort=10 velocity=1.0
- added joint right_finger_joint: type revolute, parent wheeltec_gripper_chaise, child right_finger, origin xyz=0.071485 0.047224 -0.01437 rpy=0 0 0.7298, axis -2.5729E-05 0.080001 -0.99679, limit lower=0 upper=0.7298 effort=10 velocity=1.0, mimic joint=left_finger_joint multiplier=1 offset=0
- added joint wheeltec_gripper_base_link_joint: type fixed, parent wheeltec_gripper_base_link, child wheeltec_gripper_chaise, origin xyz=-0.005 0 0.0272 rpy=0 -1.5707963267948966 0
- added joint wheeltec_gripper_center_joint: type fixed, parent wheeltec_gripper_chaise, child wheeltec_gripper_center, origin xyz=0 0 0 rpy=0 0 0, axis 0 0 0.001
- added joint wheeltec_gripper_end_link_joint: type fixed, parent ar3_end_link, child wheeltec_gripper_base_link
- joint camera_joint: origin xyz=0 -0.55 1.0 rpy=0 1.5707963267948966 0 -> xyz=-0.1 -0.35 0.75 rpy=0 1.5707963267948966 0
- joint camera_link_joint: origin xyz=0.010600000000000002 0.0175 0.0125 rpy=0 0 0 -> xyz=0 0.0175 0.0125 rpy=0 0 0
